Commit message: Add mass and collision in robot

File: src/robot/urdf/robot.urdf (robot description, URDF)
Before this commit: robot myrobot, 3 links, 2 joints
Links:
- link base_link: mass None -> 10; geometry collision cylinder length=0.3 radius=0.2; visual cylinder length=0.3 radius=0.4
- link left_wheel: mass None -> 10; geometry collision cylinder length=0.1 radius=0.2; visual cylinder length=0.1 radius=0.2
- link right_wheel: mass None -> 10; geometry collision cylinder length=0.1 radius=0.2; visual cylinder length=0.1 radius=0.2
Joints:
- joint base_to_left_wheel: axis (none) -> 0 1 0; type fixed -> continuous
- joint base_to_right_wheel: axis (none) -> 0 1 0; type fixed -> continuous

Commit message: create xacro file in uref

File: src/robot/urdf/robot.urdf (robot description, URDF)
Before this commit: robot myrobot, 3 links, 2 joints
Links:
- link base_link: mass 10 -> None
- link left_wheel: mass 10 -> None; geometry 
- link right_wheel: mass 10 -> None; geometry 
