Commit message: Not Success

File: src/robot/urdf/meterial.xacro (robot description, xacro)
@@ -1,17 +1,21 @@
 <?xml version="1.0" ?>
 <robot name="myrobot" xmlns:xacro="https://www.ros.org/wiki/xacro">
-  <xacro:macro name="default_wheel_visual_collision">
+  <xacro:macro name="default_wheel_visual_collision" params="reflect">
  <visual>
             <geometry>
-                <cylinder length="0.1" radius="0.2"/>
+                <cylinder length="0.1" radius="0.5"/>
             </geometry>
             <material name="blue"/>
-            <origin rpy="0 1.57075 1.57075" xyz="0 0 0"/>
+            <origin rpy="0 1.57075 1.57075" xyz="0 ${reflect} 0"/>
         </visual>
         <collision>
             <geometry>
-                <cylinder length="0.1" radius="0.2"/>
+                <cylinder length="0.1" radius="0.5"/>
             </geometry>
         </collision>
+           <inertial>
+      <mass value="10" />
+      <inertia ixx="1.0" ixy="1.0" ixz="1.0" iyy="1.0" iyz="1.0" izz="1.0" />
+    </inertial>
   </xacro:macro>
 </robot>

File: src/robot/urdf/robot.urdf.xacro (robot description, xacro)
@@ -21,9 +21,9 @@
     </link>
     <link name="right_wheel">
-        <xacro:default_wheel_visual_collision />
-        <xacro:default_inertial mass="10"/>
+        <xacro:default_wheel_visual_collision reflect="0.3"/>
+        <xacro:default_inertial mass="10" />
     </link>
     <link name="left_wheel">
-        <xacro:default_wheel_visual_collision />
+        <xacro:default_wheel_visual_collision reflect="-0.3"/>
         <xacro:default_inertial mass="10"/>
     </link>
@@ -40,10 +40,19 @@
         <axis xyz="0 1 0"/>
     </joint>
-    <transmission name="${prefix}_wheel_trans">
+    <transmission name="right_wheel_trans">
       <type>transmission_interface/SimpleTransmission</type>
-      <actuator name="${prefix}_wheel_motor">
+      <actuator name="right_wheel_motor">
         <mechanicalReduction>1</mechanicalReduction>
       </actuator>
-      <joint name="$base_to_${prefix}_wheel">
+      <joint name="base_to_right_wheel">
+        <hardwareInterface>VelocityJointInterface</hardwareInterface>
+      </joint>
+    </transmission>
+    <transmission name="left_wheel_trans">
+      <type>transmission_interface/SimpleTransmission</type>
+      <actuator name="left_wheel_motor">
+        <mechanicalReduction>1</mechanicalReduction>
+      </actuator>
+      <joint name="base_to_$left_wheel">
         <hardwareInterface>VelocityJointInterface</hardwareInterface>
       </joint>
@@ -54,5 +63,12 @@
     </plugin>
   </gazebo>
-  <gazebo reference="${prefix}_wheel">
+  <gazebo reference="left_wheel">
+      <mu1 value="200.0"/>
+      <mu2 value="100.0"/>
+      <kp value="10000000.0" />
+      <kd value="1.0" />
+      <material>Gazebo/Grey</material>
+    </gazebo>
+    <gazebo reference="right_wheel">
       <mu1 value="200.0"/>
       <mu2 value="100.0"/>

Commit message: Add robot part 1

File: src/robot/urdf/meterial.xacro (robot description, xacro)
@@ -14,8 +14,8 @@
             </geometry>
         </collision>
-           <inertial>
+           <!-- <inertial>
       <mass value="10" />
       <inertia ixx="1.0" ixy="1.0" ixz="1.0" iyy="1.0" iyz="1.0" izz="1.0" />
-    </inertial>
+    </inertial> -->
   </xacro:macro>
 </robot>
